File: hardware/Face.brd (EAGLE design)
At the start: 100 x 80 mm, 189 parts

Commit message: Removing dependence on Sparkfun-LED
Parts:
- LED10, LED100, LED101, LED102, LED103, LED104, LED105, LED106, LED107, LED108, LED109, LED11, LED110, LED111, LED112, LED113, LED114, LED115, LED116, LED117, LED118, LED119, LED12, LED120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: device SparkFun-LED:LED-0603 -> Customs:LED-0603
